Commit message: transmission carrellino e pendolo

File: modello/urdf/pendolo_inv.urdf.xacro (robot description, xacro)
@@ -10,4 +10,6 @@
         <color rgba="1 1 1 0.5"/>
     </material>
+<!-- Questo è il link base nella terna base_link rispetto alla quale vengono definite tutte le altre terne
+tale elemento ha il solo scopo di esser di riferimento rispetto al robot mobile -->
     <link name="base_link">
         <visual>
@@ -28,5 +30,5 @@
     </link>
     <link name="carrellino">
-        <!--        base link è la terna collegata a questo giunto-->
+        <!--questo è il solo elemento mobile attuato-->
         <visual>
             <origin rpy="0 0 0" xyz="0 0 0"/>
@@ -52,4 +54,14 @@
         <origin rpy="0 0 0" xyz="0 0 0"/>
     </joint>
+<transmission name="carrellino_trans">
+    <type>transmission_interface/SimpleTransmission</type>
+    <actuator name="carrellino_motor">
+      <hardwareInterface>hardware_interface/PositionJointInterface</hardwareInterface>
+      <mechanicalReduction>1</mechanicalReduction>
+    </actuator>
+    <joint name="base_carrellino">
+      <hardwareInterface>hardware_interface/PositionJointInterface</hardwareInterface>
+    </joint>
+  </transmission>
     <link name="left_wheel">
         <visual>
@@ -132,3 +144,18 @@
         <origin rpy="0 0 0" xyz="0 0 0.1"/>
     </joint>
+    <transmission name="pendolo_trans">
+        <type>transmission_interface/SimpleTransmission</type>
+        <actuator name="pendolo_motor">
+            <hardwareInterface>hardware_interface/EffortJointInterface</hardwareInterface>
+            <mechanicalReduction>1</mechanicalReduction>
+        </actuator>
+        <joint name="pendolo_joint">
+             <hardwareInterface>hardware_interface/EffortJointInterface</hardwareInterface>
+        </joint>
+    </transmission>
+    <gazebo>
+        <plugin name="gazebo_ros_control" filename="libgazebo_ros_control.so">
+            <robotNamespace>/</robotNamespace>
+        </plugin>
+    </gazebo>
 </robot>

Commit message: Controllo in velocità tramite nodo publisher.py

File: modello/urdf/pendolo_inv.urdf.xacro (robot description, xacro)
@@ -12,4 +12,9 @@
 <!-- Questo è il link base nella terna base_link rispetto alla quale vengono definite tutte le altre terne
 tale elemento ha il solo scopo di esser di riferimento rispetto al robot mobile -->
+    <link name="world"/>
+    <joint name="fixed" type="fixed">
+        <parent  link="world"/>
+        <child link="base_link"/>
+    </joint>
     <link name="base_link">
         <visual>
@@ -51,5 +56,5 @@
         <parent link="base_link"/>
         <child link="carrellino"/>
-        <limit effort="1000.0" lower="-0.5" upper="0.5" velocity="0.5"/>
+        <limit effort="999999.0" lower="-50" upper="50" velocity="500"/>
         <origin rpy="0 0 0" xyz="0 0 0"/>
     </joint>
@@ -57,9 +62,9 @@
     <type>transmission_interface/SimpleTransmission</type>
     <actuator name="carrellino_motor">
-      <hardwareInterface>hardware_interface/PositionJointInterface</hardwareInterface>
+      <hardwareInterface>hardware_interface/VelocityJointInterface</hardwareInterface>
       <mechanicalReduction>1</mechanicalReduction>
     </actuator>
     <joint name="base_carrellino">
-      <hardwareInterface>hardware_interface/PositionJointInterface</hardwareInterface>
+      <hardwareInterface>hardware_interface/VelocityJointInterface</hardwareInterface>
     </joint>
   </transmission>
@@ -132,11 +137,13 @@
         </collision>
         <inertial>
-            <mass value="3"/>
-            <inertia ixx="1.0" ixy="0.0" ixz="0.0" iyy="1.0" iyz="0.0" izz="1.0"/>
+            <mass value="0.02"/>
+            <inertia ixx="0.0007" ixy="0.0" ixz="0.0" iyy="0.0007" iyz="0.0" izz="0.000013"/>
+            <origin xyz="0 0 0.2" rpy="0 0 0 "/>
         </inertial>
     </link>
     <joint name="pendolo_joint" type="revolute">
-        <limit effort="1000.0" lower="-1.5707" upper="1.5707" velocity="0.5"/>
-        <axis rpy="0 0 0" xyz="0 1 0"/>
+        <limit effort="1000.0" lower="-1.1" upper="1.1"  velocity="100"/>
+        <dynamics damping="0.001" friction="0.0"/>
+        <axis rpy="0 0 0" xyz="0 1 0.1"/>
         <parent link="carrellino"/>
         <child link="pendolo"/>

Commit message: MPC con solver lento

File: modello/urdf/pendolo_inv.urdf.xacro (robot description, xacro)
@@ -49,5 +49,5 @@
         </collision>
         <inertial>
-            <mass value="10"/>
+            <mass value="1"/>
             <inertia ixx="1.0" ixy="0.0" ixz="0.0" iyy="1.0" iyz="0.0" izz="1.0"/>
         </inertial>
@@ -56,5 +56,5 @@
         <parent link="base_link"/>
         <child link="carrellino"/>
-        <limit effort="999999.0" lower="-50" upper="50" velocity="500"/>
+        <limit effort="999999.0" lower="-10" upper="10" velocity="5000"/>
         <origin rpy="0 0 0" xyz="0 0 0"/>
     </joint>
@@ -62,9 +62,9 @@
     <type>transmission_interface/SimpleTransmission</type>
     <actuator name="carrellino_motor">
-      <hardwareInterface>hardware_interface/VelocityJointInterface</hardwareInterface>
+      <hardwareInterface>hardware_interface/EffortJointInterface</hardwareInterface>
       <mechanicalReduction>1</mechanicalReduction>
     </actuator>
     <joint name="base_carrellino">
-      <hardwareInterface>hardware_interface/VelocityJointInterface</hardwareInterface>
+      <hardwareInterface>hardware_interface/EffortJointInterface</hardwareInterface>
     </joint>
   </transmission>
@@ -124,24 +124,24 @@
         <visual>
             <!--            origin mi indica dove rispetto alla struttura del pendolo fisso gli assi cartesiani-->
-            <origin rpy="0 0 0" xyz="0 0 0.2"/>
+            <origin rpy="0 0 0" xyz="0 0 0.75"/>
             <geometry>
-                <cylinder length="0.4" radius="0.035"/>
+                <cylinder length="1.5" radius="0.035"/>
             </geometry>
             <material name="violetto"/>
         </visual>
         <collision>
-            <origin rpy="0 0 0" xyz="0 0 0.2"/>
+            <origin rpy="0 0 0" xyz="0 0 0.75"/>
             <geometry>
-                <cylinder length="0.4" radius="0.035"/>
+                <cylinder length="1.5" radius="0.035"/>
             </geometry>
         </collision>
         <inertial>
-            <mass value="0.02"/>
-            <inertia ixx="0.0007" ixy="0.0" ixz="0.0" iyy="0.0007" iyz="0.0" izz="0.000013"/>
-            <origin xyz="0 0 0.2" rpy="0 0 0 "/>
+            <mass value="0.1"/>
+            <inertia ixx="0.019" ixy="0.0" ixz="0.0" iyy="0.019" iyz="0.0" izz="0.0175"/>
+            <origin xyz="0 0 0.75" rpy="0 0 0 "/>
         </inertial>
     </link>
     <joint name="pendolo_joint" type="revolute">
-        <limit effort="1000.0" lower="-1.1" upper="1.1"  velocity="100"/>
+        <limit effort="1000.0" lower="-1.0" upper="1.0"  velocity="100"/>
         <dynamics damping="0.001" friction="0.0"/>
         <axis rpy="0 0 0" xyz="0 1 0.1"/>

Commit message: MPC con dinamica corretta

File: modello/urdf/pendolo_inv.urdf.xacro (robot description, xacro)
@@ -56,6 +56,6 @@
         <parent link="base_link"/>
         <child link="carrellino"/>
-        <limit effort="999999.0" lower="-10" upper="10" velocity="5000"/>
-        <origin rpy="0 0 0" xyz="0 0 0"/>
+        <limit effort="999999.0" lower="-50" upper="50" velocity="5000"/>
+        <origin rpy="0 0 0" xyz="0 0 1"/>
     </joint>
 <transmission name="carrellino_trans">
@@ -124,26 +124,26 @@
         <visual>
             <!--            origin mi indica dove rispetto alla struttura del pendolo fisso gli assi cartesiani-->
-            <origin rpy="0 0 0" xyz="0 0 0.75"/>
+            <origin rpy="0 0 0" xyz="0 0 0.25"/>
             <geometry>
-                <cylinder length="1.5" radius="0.035"/>
+                <cylinder length="0.5" radius="0.035"/>
             </geometry>
             <material name="violetto"/>
         </visual>
         <collision>
-            <origin rpy="0 0 0" xyz="0 0 0.75"/>
+            <origin rpy="0 0 0" xyz="0 0 0.25"/>
             <geometry>
-                <cylinder length="1.5" radius="0.035"/>
+                <cylinder length="0.5" radius="0.035"/>
             </geometry>
         </collision>
         <inertial>
             <mass value="0.1"/>
-            <inertia ixx="0.019" ixy="0.0" ixz="0.0" iyy="0.019" iyz="0.0" izz="0.0175"/>
-            <origin xyz="0 0 0.75" rpy="0 0 0 "/>
+            <inertia ixx="0.0021" ixy="0.0" ixz="0.0" iyy="0.0021" iyz="0.0" izz="0.000061"/>
+            <origin xyz="0 0 0.25" rpy="0 0 0 "/>
         </inertial>
     </link>
-    <joint name="pendolo_joint" type="revolute">
-        <limit effort="1000.0" lower="-1.0" upper="1.0"  velocity="100"/>
+    <joint name="pendolo_joint" type="continuous">
+        <limit effort="1000.0" velocity="10000"/>
         <dynamics damping="0.001" friction="0.0"/>
-        <axis rpy="0 0 0" xyz="0 1 0.1"/>
+        <axis xyz="0 1 0"/>
         <parent link="carrellino"/>
         <child link="pendolo"/>
